Commit message: lasers are added

File: ros/src/irobotcreate2ros/iRobot/iRobot.urdf (robot description, URDF)
Before this commit: robot iRobot, 10 links, 9 joints
Links:
- added link hokuyo_link, mass 1e-5; collision cylinder length=0.12 radius=0.015; visual cylinder length=0.12 radius=0.015
- added link hokuyo_link_2, mass 1e-5; collision cylinder length=0.12 radius=0.015; visual cylinder length=0.12 radius=0.015
- link camera_link: geometry collision box size=0.02 0.08 0.11; visual box size=0.02 0.08 0.11
Joints:
- added joint hokuyo_laser_joint: type fixed, parent base_link, child hokuyo_link, origin xyz=0.08 0.09 0.1 rpy=0 -0.1 3.11, axis 0 0 0
- added joint hokuyo_laser_joint_2: type fixed, parent base_link, child hokuyo_link_2, origin xyz=0.08 -0.09 0.1 rpy=0 -0.1 3.45, axis 0 0 0

File: ros/src/irobotcreate2ros/model/camera.urdf.xacro (robot description, xacro)
@@ -13,5 +13,5 @@
                 <origin xyz="0 0 0" rpy="0 0 0"/>
                 <geometry>
-                    <box size="0.02 0.08 0.05"/>
+                    <box size="0.02 0.08 0.11"/>
                 </geometry>
             </collision>
@@ -19,5 +19,5 @@
                 <origin xyz="0 0 0" rpy="0 0 0"/>
                 <geometry>
-                    <box size="0.02 0.08 0.05"/>
+                    <box size="0.02 0.08 0.11"/>
                 </geometry>
                 <material name="iRobot/Green"/>
@@ -35,6 +35,6 @@
                     <horizontal_fov>1.3962634</horizontal_fov>
                     <image>
-                        <width>800</width>
-                        <height>600</height>
+                        <width>640</width>
+                        <height>480</height>
                         <format>R8G8B8</format>
                     </image>

File: ros/src/irobotcreate2ros/model/hokuyo.urdf.xacro (robot description, xacro)
@@ -3,14 +3,14 @@
 <xacro:macro name="hokuyo_laser" params="xyz rpy parent">
     <joint name="hokuyo_laser_joint" type="fixed">
-        <axis xyz="0 0 1" />
+        <axis xyz="0 0 0" />
         <origin xyz="${xyz}" rpy="${rpy}"/>
         <parent link="${parent}"/>
-        <child link="hokuyo_laser_link"/>
+        <child link="hokuyo_link"/>
     </joint>
-    <link name="hokuyo_laser_link">
+    <link name="hokuyo_link">
         <collision>
             <origin xyz="0 0 0" rpy="0 0 0"/>
             <geometry>
-                <cylinder length="0.04" radius="0.045"/>
+                <cylinder length="0.12" radius="0.015"/>l
             </geometry>
         </collision>
@@ -18,5 +18,5 @@
             <origin xyz="0 0 0" rpy="0 0 0"/>
             <geometry>
-                <cylinder length="0.04" radius="0.045"/>
+                <cylinder length="0.12" radius="0.015"/>
             </geometry>
             <material name="iRobot/LightBlue"/>
@@ -28,5 +28,5 @@
         </inertial>
     </link>
-    <gazebo reference="hokuyo_laser_link">
+    <gazebo reference="hokuyo_link">
         <gravity>true</gravity>
         <sensor type="ray" name="head_hokuyo_sensor">
@@ -37,8 +37,8 @@
                 <scan>
                     <horizontal>
-                        <samples>360</samples>
+                        <samples>2</samples>
                         <resolution>1</resolution>
-                        <min_angle>-3.14159</min_angle>
-                        <max_angle>3.14159</max_angle>
+                        <min_angle>-3.14</min_angle>
+                        <max_angle>3.14</max_angle>
                     </horizontal>
                 </scan>
@@ -55,7 +55,6 @@
             </ray>
             <plugin name="gazebo_ros_head_hokuyo_controller" filename="libgazebo_ros_laser.so">
-                <robotNamespace></robotNamespace>
-                <topicName>laser_scan</topicName>
-                <frameName>hokuyo_laser_link</frameName>
+                <topicName>/laser_scan</topicName>
+                <frameName>hokuyo_link</frameName>
             </plugin>
         </sensor>

File: ros/src/irobotcreate2ros/model/iRobot.urdf.xacro (robot description, xacro)
@@ -7,5 +7,6 @@
   <xacro:include filename="$(find irobotcreate2)/model/shelf.urdf.xacro"/>
   <xacro:include filename="$(find irobotcreate2)/gazebo/iRobot.gazebo.xacro"/>
-  <!--<xacro:include filename="$(find irobotcreate2)/model/hokuyo.urdf.xacro"/>-->
+  <xacro:include filename="$(find irobotcreate2)/model/hokuyo.urdf.xacro"/>
+  <xacro:include filename="$(find irobotcreate2)/model/hokuyo_v2.urdf.xacro"/>
   <xacro:include filename="$(find irobotcreate2)/model/imu.urdf.xacro"/>
   <xacro:include filename="$(find irobotcreate2)/model/camera.urdf.xacro"/>
@@ -122,9 +123,14 @@
         </collision>
     </link>
-    <!-- Laser link and plugin -->
-    <!--<xacro:hokuyo_laser xyz="0 0 ${0.04 + 0.02}"
-                  rpy="0 0 0"
+    <!-- Laser link and plugin v1 -->
+    <xacro:hokuyo_laser xyz="0.08 0.09 ${0.04 + 0.02 + 0.04}"
+                  rpy="0 -0.1 3.11"
                   parent="base_link">
-    </xacro:hokuyo_laser>-->
+    </xacro:hokuyo_laser>
+    <!-- Laser link and plugin v2 -->
+    <xacro:hokuyo_laser_2 xyz="0.08 -0.09 ${0.04 + 0.02 + 0.04}"
+                  rpy="0 -0.1 3.45"
+                  parent="base_link">
+    </xacro:hokuyo_laser_2>
     <!--Imu link and plugin-->
     <xacro:imu_sensor xyz="-0.1 0 ${0.04 + 0.01}"

Commit message: 2 camera is added

File: ros/src/irobotcreate2ros/iRobot/iRobot.urdf (robot description, URDF)
Before this commit: robot iRobot, 12 links, 11 joints
Links:
- added link box, mass 1; collision box size=0.01 0.01 0.5; visual box size=0.01 0.01 0.5
- added link camera_up_link, mass 0.0001; collision box size=0.02 0.05 0.05; visual box size=0.02 0.05 0.05
Joints:
- added joint box: type fixed, parent base_link, child box, origin xyz=-0.10 0 0.25 rpy=0 0 0
- added joint camera_up_sensor_joint: type fixed, parent base_link, child camera_up_link, origin xyz=-0.08 0 0.5 rpy=0 1.4 0, axis 0 1 0
- joint camera_sensor_joint: origin xyz=0 0 0.1 rpy=0 0 0 -> xyz=0.08 0 0.1 rpy=0 0 0

File: ros/src/irobotcreate2ros/model/iRobot.urdf.xacro (robot description, xacro)
@@ -11,4 +11,5 @@
   <xacro:include filename="$(find irobotcreate2)/model/imu.urdf.xacro"/>
   <xacro:include filename="$(find irobotcreate2)/model/camera.urdf.xacro"/>
+  <xacro:include filename="$(find irobotcreate2)/model/camera_up.urdf.xacro"/>
   <xacro:include filename="$(find irobotcreate2)/model/bumper.urdf.xacro"/>
   <xacro:property name="pi" value="3.1415926535897931"/>
@@ -44,4 +45,29 @@
             <geometry>
                 <cylinder length="0.08" radius="0.17"/>
+            </geometry>
+        </collision>
+    </link>
+    <joint name="box" type="fixed">
+        <origin xyz="-0.10 0 0.25" rpy="0 0 0" />
+        <parent link="base_link"/>
+        <child link="box"/>
+    </joint>
+    <link name="box">
+        <inertial>
+            <origin xyz="0 0 0" rpy="0 0 0"/>
+            <mass value="1"/>
+             <inertia ixx="${1/12*10*3*0.17*0.17+1/12*5*3*0.08*0.08}" ixy="0.0" ixz="0.0" iyy="${1/12*10*3*0.17*0.17+1/12*5*3*0.08*0.08}" iyz="0.0" izz="${1/2*10*0.17*0.17}"/>
+        </inertial>
+        <visual>
+            <origin xyz="0 0 0" rpy="0 0 0"/>
+            <geometry>
+                <box size="0.01 0.01 0.5"/>
+            </geometry>
+            <material name="iRobot/Black"/>
+        </visual>
+        <collision name="box">
+            <origin xyz="0 0 0" rpy="0 0 0"/>
+            <geometry>
+                <box size="0.01 0.01 0.5"/>
             </geometry>
         </collision>
@@ -139,8 +165,13 @@
     </xacro:imu_sensor>
     <!--Camera link and plugin-->
-    <xacro:camera_sensor xyz="0 0 ${0.04 + 0.02 + 0.04}"
+    <xacro:camera_sensor xyz="0.08 0 ${0.04 + 0.02 + 0.04}"
                   rpy="0 0 0"
                   parent="base_link">
     </xacro:camera_sensor>
+    <!--Camera up link and plugin-->
+    <xacro:camera_up_sensor xyz="-0.08 0 0.5"
+                  rpy="0 1.4 0"
+                  parent="base_link">
+    </xacro:camera_up_sensor>
     <!--Bumper link and plugin-->
     <xacro:bumper_sensor xyz="0 0 0"
